File: Hardware/Projekt/ServoShield/ServoShield_Protorype.sch (EAGLE design)
At the start: 66 parts, among them IC0 74HCT595D, IC1 74HCT595D, IC2 74HCT595D, IC3 74HCT595D, Q1 16MHz

Commit message: Rearranged Parts
Parts:
- removed 3TO5: 74HCT541DW, 74xx-eu:74HCT541DW
- removed 5TO3_VERORGUNG_äNDERN: 74AC541DW, 74xx-eu:74AC541DW
Connections:
- net +5V/1: now also JP1.6; no longer JP1.1
- net +5V/2: now also JP1.1; no longer JP1.5
- net GND: now also JP1.3, JP1.5; no longer 3TO5A.G1, 3TO5A.G2, 5TO3_VERORGUNG_äNDERNA.G1, 5TO3_VERORGUNG_äNDERNA.G2, JP1.4, JP1.6
- net VCC: now also JP1.4; no longer JP1.3

Commit message: Changed Pinheader and routed all signals
It is not possible to connect 8 servos on one 3x8 pinheader. The servo connectors are to wide. All 3x8 pinheader where changed for 2 3x4 pinheaders.
Parts:
- removed SGND0, SGND1, SGND2, SGND3, SVCC0, SVCC1, SVCC2, SVCC3: (no value), pinhead:PINHD-1X8
- added LED1: GN_2V, led:LED3MM
- added R39: 1k5, rcl:R-EU_R0805
- added SD-4, SD-5, SD-6, SD-7: (no value), pinhead:PINHD-1X4
- added V_GND0, V_GND1, V_GND2, V_GND3, V_GND4, V_GND5, V_GND6, V_GND7: (no value), pinhead:PINHD-2X4
- JP1: device pinhead:PINHD-1X6/90 -> pinhead:PINHD-1X6
- SD-0, SD-1, SD-2, SD-3: device pinhead:PINHD-1X8 -> pinhead:PINHD-1X4
Connections:
- removed net N$23: ATMEGA328.PC1(ADC1/PCINT9)
- new net LED: ATMEGA328.PD7(AIN1/PCINT23), R39.1
- new net N$85: LED1.A, R39.2
- net +5V/1: now also V_GND0.1, V_GND0.3, V_GND0.5, V_GND0.7, V_GND1.1, V_GND1.3, V_GND1.5, V_GND1.7, V_GND2.1, V_GND2.3, V_GND2.5, V_GND2.7, V_GND3.1, V_GND3.3, V_GND3.5, V_GND3.7; no longer SVCC0.1, SVCC0.2, SVCC0.3, SVCC0.4, SVCC0.5, SVCC0.6, SVCC0.7, SVCC0.8, SVCC1.1, SVCC1.2, SVCC1.3, SVCC1.4, SVCC1.5, SVCC1.6, SVCC1.7, SVCC1.8
- net +5V/2: now also V_GND4.1, V_GND4.3, V_GND4.5, V_GND4.7, V_GND5.1, V_GND5.3, V_GND5.5, V_GND5.7, V_GND6.1, V_GND6.3, V_GND6.5, V_GND6.7, V_GND7.1, V_GND7.3, V_GND7.5, V_GND7.7; no longer SVCC2.1, SVCC2.2, SVCC2.3, SVCC2.4, SVCC2.5, SVCC2.6, SVCC2.7, SVCC2.8, SVCC3.1, SVCC3.2, SVCC3.3, SVCC3.4, SVCC3.5, SVCC3.6, SVCC3.7, SVCC3.8
- net G: now also ATMEGA328.PC1(ADC1/PCINT9); no longer ATMEGA328.PB0(ICP1/CLKO/PCINT0)
- net GND: now also LED1.C, V_GND0.2, V_GND0.4, V_GND0.6, V_GND0.8, V_GND1.2, V_GND1.4, V_GND1.6, V_GND1.8, V_GND2.2, V_GND2.4, V_GND2.6, V_GND2.8, V_GND3.2, V_GND3.4, V_GND3.6, V_GND3.8, V_GND4.2, V_GND4.4, V_GND4.6, V_GND4.8, V_GND5.2, V_GND5.4, V_GND5.6, V_GND5.8, V_GND6.2, V_GND6.4, V_GND6.6, V_GND6.8, V_GND7.2, V_GND7.4, V_GND7.6, V_GND7.8; no longer SGND0.1, SGND0.2, SGND0.3, SGND0.4, SGND0.5, SGND0.6, SGND0.7, SGND0.8, SGND1.1, SGND1.2, SGND1.3, SGND1.4, SGND1.5, SGND1.6, SGND1.7, SGND1.8, SGND2.1, SGND2.2, SGND2.3, SGND2.4, SGND2.5, SGND2.6, SGND2.7, SGND2.8, SGND3.1, SGND3.2, SGND3.3, SGND3.4, SGND3.5, SGND3.6, SGND3.7, SGND3.8
- net N$29: now also SD-1.1; no longer SD-0.5
- net N$30: now also SD-1.2; no longer SD-0.6
- net N$31: now also SD-1.3; no longer SD-0.7
- net N$32: now also SD-1.4; no longer SD-0.8
- net N$34: now also SD-2.1; no longer SD-1.1
- net N$43: now also SD-2.2; no longer SD-1.2
- net N$44: now also SD-2.3; no longer SD-1.3
- net N$45: now also SD-2.4; no longer SD-1.4
- net N$46: now also SD-3.1; no longer SD-1.5
- net N$47: now also SD-3.2; no longer SD-1.6
- net N$48: now also SD-3.3; no longer SD-1.7
- net N$49: now also SD-3.4; no longer SD-1.8
- net N$60: now also SD-4.1; no longer SD-2.1
- net N$61: now also SD-4.2; no longer SD-2.2
- net N$62: now also SD-4.3; no longer SD-2.3
- net N$63: now also SD-4.4; no longer SD-2.4
- net N$64: now also SD-5.1; no longer SD-2.5
- net N$65: now also SD-5.2; no longer SD-2.6
- net N$66: now also SD-5.3; no longer SD-2.7
- net N$67: now also SD-5.4; no longer SD-2.8
- net N$76: now also SD-6.1; no longer SD-3.1
- net N$77: now also SD-6.2; no longer SD-3.2
- net N$78: now also SD-6.3; no longer SD-3.3
- net N$79: now also SD-6.4; no longer SD-3.4
- net N$80: now also SD-7.1; no longer SD-3.5
- net N$81: now also SD-7.2; no longer SD-3.6
- net N$82: now also SD-7.3; no longer SD-3.7
- net N$83: now also SD-7.4; no longer SD-3.8
- net N$9: now also ATMEGA328.PB0(ICP1/CLKO/PCINT0); no longer ATMEGA328.PD7(AIN1/PCINT23)
