File: Hardware/Projekt/ServoShield_v2/ServoShield_v2_2.brd (EAGLE design)
At the start: 100 x 80 mm, 60 parts, among them IC1 ATMEGA644A, Q1 8MHz

Commit message: Added connectors for power and finished routing
Parts:
- removed JP1: (no value), pinhead:1X06
- added C5, C6, C7, C8: 100nF, resistor:C0805
- added X1, X2, X3: MST2V, PHO508E:MSTBV2
- moved POLULU_MINIMU-9_V5 42.8 mm to (52.7, 27.3)
- moved R28 3.59 mm to (8.89, 33.0), turned to 0 degrees
- moved R27 2.54 mm to (8.89, 40.6)
- moved R39 2.54 mm to (8.89, 45.7)
- moved LED1 2.54 mm to (5.08, 45.7), turned to 270 degrees
- moved LED2 2.54 mm to (5.08, 40.6), turned to 270 degrees
- moved LED3 2.54 mm to (5.08, 35.6), turned to 270 degrees
- moved R1 1.27 mm to (3.81, 16.5)
- moved C3 1.27 mm to (14.6, 14.6)
- moved S1 0.63 mm to (6.35, 10.8)
Connections:
- net +5V/1: now also C7.1, X2.2; no longer JP1.1
- net +5V/2: now also C8.1, X3.2; no longer JP1.6
- net GND: now also C5.1, C6.1, C7.2, C8.2, X1.1, X2.1, X3.1; no longer JP1.2, JP1.3, JP1.5
- net VCC: now also C5.2, C6.2, X1.2; no longer JP1.4
Routing:
- net SCL: track 41.9 -> 61.7 mm, vias 2 -> 1
- net SDA: track 45.9 -> 64.3 mm, vias 2 -> 1
- net +5V/2: track 0.00 -> 4.99 mm
- net +5V/1: track 0.00 -> 3.83 mm
- net LED_1: track 23.7 -> 20.5 mm
- net LED_2: track 27.1 -> 24.6 mm
- net LED_3: track 31.1 -> 28.6 mm
- net N$28: track 3.01 -> 5.34 mm
- net !RST: track 39.7 -> 40.9 mm
- net SERVO_12: track 24.9 -> 26.0 mm
- net SCK: track 20.2 -> 21.2 mm
- net MISO: track 17.3 -> 18.4 mm
- net VCC: track 45.4 -> 44.4 mm, vias 6 -> 4
- net N$27: track 3.01 -> 3.94 mm
- net N$85: track 3.01 -> 3.94 mm

Commit message: Minor changes
Parts:
- removed C7, C8: 100nF, resistor:C0805
Connections:
- net +5V/1: no longer C7.1
- net +5V/2: no longer C8.1
- net GND: no longer C7.2, C8.2
Routing:
- net +5V/2: track 4.99 -> 0.95 mm
- net +5V/1: track 3.83 -> 1.59 mm
Changed lines of the file:
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@@
 <element name="C5" library="resistor" package="C0805" value="100nF" x="56.515" y="26.67" rot="MR90"/>
 <element name="C6" library="resistor" package="C0805" value="100nF" x="15.24" y="19.05" rot="MR0"/>
-<element name="C7" library="resistor" package="C0805" value="100nF" x="57.785" y="38.1" rot="MR270"/>
-<element name="C8" library="resistor" package="C0805" value="100nF" x="57.15" y="13.97" rot="MR270"/>
 </elements>
 <signals>
@@
 <contactref element="C5" pad="1"/>
 <contactref element="C6" pad="1"/>
-<contactref element="C8" pad="2"/>
-<contactref element="C7" pad="2"/>
 <contactref element="X2" pad="1"/>
 </signal>
@@
 </polygon>
 <contactref element="X2" pad="2"/>
-<contactref element="C7" pad="1"/>
-<wire x1="57.785" y1="39.05" x2="59.375" y2="40.64" width="0.4064" layer="16"/>
 <wire x1="59.375" y1="40.64" x2="60.96" y2="40.64" width="0.4064" layer="16"/>
 </signal>
@@
 </polygon>
 <contactref element="X3" pad="2"/>
-<contactref element="C8" pad="1"/>
-<wire x1="57.15" y1="14.92" x2="60.01" y2="17.78" width="0.4064" layer="16"/>
 <wire x1="60.01" y1="17.78" x2="60.96" y2="17.78" width="0.4064" layer="16"/>
 </signal>
