File: Hardware/Projekt/ServoShield_v2/ServoShield_v2_3.brd (EAGLE design)
At the start: 100 x 80 mm, 64 parts, among them IC1 ATMEGA644A, Q1 8MHz, X1 MST2V, X2 MST2V, X3 MST2V

Commit message: Changed power connectors and added vias for Servo vcc lines
Parts:
- removed X1, X2, X3: MST2V, PHO508E:MSTBV2
- added X4, X5, X6: MCV2, con-phoenix_3.81_mcv:MCV2
- moved C5 1.27 mm to (57.1, 26.7), turned to 90 degrees
- moved USB_RASP 1.27 mm to (14.0, 6.35)
- moved R6 1.27 mm to (10.2, 3.81)
- moved C3 1.27 mm to (14.6, 13.3)
Connections:
- net +5V/1: now also X4.2; no longer X2.2
- net +5V/2: now also X6.1; no longer X3.2
- net GND: now also X4.1, X5.1, X6.2; no longer X1.1, X2.1, X3.1
- net VCC: now also X5.2; no longer X1.2
Routing:
- net +5V/2: track 0.95 -> 45.5 mm, vias 0 -> 5
- net +5V/1: track 1.59 -> 45.5 mm, vias 0 -> 5
- net GND: track 96.6 -> 113.4 mm, vias 2 -> 3
- net VCC: track 42.7 -> 44.3 mm
