File: Hardware/Projekt/ServoShield_v2/Raspberry_PI_Servo_Hat_v1.brd (EAGLE design)
At the start: 100 x 80 mm, 64 parts, among them IC1 ATMEGA644A, Q2 8MHz, X4 MCV2, X5 MCV2, X6 MCV2

Commit message: Minor changes in Servo board and created a release version
Parts:
- removed C5: 100nF, resistor:C0805
- moved R8 2.29 mm to (36.8, 41.3), turned to 90 degrees
- moved R28 0.90 mm to (8.26, 33.7), turned to 90 degrees
Connections:
- removed net N$33: POLULU_MINIMU-9_V5.5
- new net VDD: JP3.1, POLULU_MINIMU-9_V5.5
- net GND: no longer C5.1, JP3.39
- net VCC: no longer C5.2, POLULU_MINIMU-9_V5.4
Routing:
- net VDD: track 0.00 -> 66.5 mm, vias 0 -> 1
- net VCC: track 61.9 -> 52.5 mm, vias 9 -> 8
- net SDA: track 64.7 -> 66.0 mm
- net SCL: track 61.8 -> 62.7 mm
- net SERVO_6: track 9.61 -> 10.4 mm
- net LED_1: track 20.5 -> 21.3 mm
Other:
- board text added: "Raspberry PI Servo Hat v1"
- board text removed: "RASPI-Servo-Shield"
