File: Hardware/Projekt/LegController/leg_controller.brd (EAGLE design)
At the start: 49.2 x 47 mm, 53 parts, among them IC1 TS1117-3.3, IC3 ATXMEGA32A4U-AU, J1 22-27-2031-03, J2 22-27-2031-03, Q1 16MHz/18pF, T1 BC847SMD, T3 BC847SMD, T4 BC847SMD, U1 INA3221AIRGVT

Commit message: Minor layout improvements
Parts:
- removed C2, C3: 10uF, rcl:C025-024X044
- added C4, C5: (no value), rcl:SMC_A
- added JP7: GPIO, pinhead:2X05
- moved PWR 20.2 mm to (36.8, 2.54), turned to 270 degrees
- moved R1.1 19.2 mm to (36.8, 5.08), turned to 0 degrees
Connections:
- net +3V3: now also C5.+, JP7.1, JP7.3, JP7.5, JP7.7, JP7.9; no longer C2.1
- net +5V/2: now also C4.+; no longer C3.1
- net GND: now also C4.-, C5.-, JP7.10, JP7.2, JP7.4, JP7.6, JP7.8; no longer C2.2, C3.2
Routing:
- net GND: track 66.7 -> 79.3 mm, vias 2 -> 3
- net +5V/2: track 16.8 -> 15.6 mm
Other:
- board text added: "BS"
- board text added: "LS"
- board text added: "Leg Controller v1.4"
- board text removed: "BOTTOM"
- board text removed: "Leg Controller v1.3"
- board text removed: "TOP"
Changed lines of the file:
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@@
 <wire x1="49.2" y1="46.98" x2="0" y2="46.98" width="0" layer="20"/>
 <wire x1="0" y1="46.98" x2="0" y2="0" width="0" layer="20"/>
-<text x="46.355" y="28.575" size="1.778" layer="1" font="vector" ratio="10" rot="R90">TOP</text>
-<text x="44.45" y="28.575" size="1.778" layer="16" font="vector" ratio="10" rot="MR90">BOTTOM</text>
-<text x="6.985" y="1.905" size="0.8128" layer="1" font="vector" ratio="20">Leg Controller v1.3</text>
+<text x="40.005" y="26.035" size="1.778" layer="1" font="vector" ratio="10">BS</text>
+<text x="46.355" y="26.035" size="1.778" layer="16" font="vector" ratio="10" rot="MR0">LS</text>
+<text x="6.985" y="1.905" size="0.8128" layer="1" font="vector" ratio="20">Leg Controller v1.4</text>
 <hole x="2.54" y="2.54" drill="2"/>
 <hole x="46.355" y="44.45" drill="2"/>
@@
 <element name="C3.3" library="rcl" package="C0805K" value="100n" x="15.24" y="30.48"/>
 <element name="IC1" library="linear" package="DPACK" value="TS1117-3.3" x="42.545" y="14.605" rot="R270"/>
-<element name="PWR" library="led" package="CHIP-LED0805" value="GREEN" x="45.085" y="20.955" rot="R180"/>
-<element name="R1.1" library="rcl" package="R0805" value="330R" x="47.625" y="20.955" rot="R270"/>
+<element name="PWR" library="led" package="CHIP-LED0805" value="GREEN" x="36.83" y="2.54" rot="R270"/>
+<element name="R1.1" library="rcl" package="R0805" value="330R" x="36.83" y="5.08"/>
 <element name="LED1" library="led" package="P-LCC4-RGB" value="RGBLED" x="23.495" y="36.83"/>
 <element name="R4" library="rcl" package="R0805" value="8" x="28.575" y="31.75" rot="R90"/>
@@
 <element name="SJ2" library="jumper" package="SJ" value="AD1" x="8.255" y="18.415" rot="MR270"/>
 <element name="SJ3" library="jumper" package="SJ" value="AD2" x="5.715" y="18.415" rot="MR270"/>
-<element name="C2" library="rcl" package="C025-024X044" value="10uF" x="41.91" y="21.59" rot="R270"/>
-<element name="C3" library="rcl" package="C025-024X044" value="10uF" x="36.83" y="3.175" rot="R270"/>
+<element name="C4" library="rcl" package="SMC_A" value="" x="39.37" y="9.525"/>
+<element name="C5" library="rcl" package="SMC_A" value="" x="39.37" y="19.685" rot="R180"/>
+<element name="JP7" library="pinhead" package="2X05" value="GPIO" x="45.085" y="36.195" rot="R90"/>
 </elements>
 <signals>
@@
 <wire x1="16.425" y1="26.365" x2="13.005" y2="26.365" width="0.4064" layer="16"/>
 <wire x1="13.005" y1="26.365" x2="12.7" y2="26.67" width="0.4064" layer="16"/>
-<wire x1="45.085" y1="19.905" x2="43.865" y2="19.905" width="0.6096" layer="1"/>
 <wire x1="21.425" y1="18.965" x2="21.425" y2="14.135" width="0.4064" layer="16"/>
 <wire x1="21.425" y1="14.135" x2="22.86" y2="12.7" width="0.4064" layer="16"/>
@@
 <wire x1="16.51" y1="26.67" x2="16.51" y2="30.21" width="0.4064" layer="1"/>
 <wire x1="16.51" y1="30.21" x2="16.24" y2="30.48" width="0.4064" layer="1"/>
-<contactref element="C3" pad="2"/>
-<contactref element="C2" pad="2"/>
-<wire x1="41.91" y1="20.32" x2="43.45" y2="20.32" width="0.6096" layer="1"/>
-<wire x1="43.45" y1="20.32" x2="43.865" y2="19.905" width="0.6096" layer="1"/>
-<wire x1="37.745" y1="16.885" x2="37.745" y2="19.965" width="1.27" layer="1"/>
-<wire x1="37.745" y1="19.965" x2="38.1" y2="20.32" width="1.27" layer="1"/>
-<wire x1="38.1" y1="20.32" x2="41.91" y2="20.32" width="1.27" layer="1"/>
+<contactref element="C4" pad="-"/>
+<contactref element="C5" pad="-"/>
+<wire x1="37.88" y1="2.54" x2="38.1" y2="2.54" width="0.4064" layer="1"/>
+<wire x1="38.1" y1="2.54" x2="39.37" y2="1.27" width="0.4064" layer="1"/>
+<wire x1="39.37" y1="1.27" x2="44.45" y2="1.27" width="0.4064" layer="1"/>
+<wire x1="44.45" y1="1.27" x2="45.72" y2="2.54" width="0.4064" layer="1"/>
+<wire x1="45.72" y1="2.54" x2="45.72" y2="3.81" width="0.4064" layer="1"/>
+<wire x1="37.745" y1="16.885" x2="37.745" y2="19.56" width="1.27" layer="1"/>
+<wire x1="37.745" y1="19.56" x2="37.87" y2="19.685" width="1.27" layer="1"/>
+<wire x1="37.87" y1="19.685" x2="37.87" y2="21.36" width="1.27" layer="1"/>
+<wire x1="37.87" y1="21.36" x2="38.1" y2="21.59" width="1.27" layer="1"/>
+<via x="38.1" y="21.59" extent="1-16" drill="0.6" diameter="1.27" shape="octagon"/>
+<wire x1="40.87" y1="9.525" x2="41.91" y2="9.525" width="1.27" layer="1"/>
+<wire x1="41.91" y1="9.525" x2="45.72" y2="5.715" width="1.27" layer="1"/>
+<wire x1="45.72" y1="5.715" x2="45.72" y2="3.81" width="1.27" layer="1"/>
+<contactref element="JP7" pad="10"/>
+<contactref element="JP7" pad="8"/>
+<contactref element="JP7" pad="6"/>
+<contactref element="JP7" pad="4"/>
+<contactref element="JP7" pad="2"/>
 </signal>
 <signal name="A0">
@@
 <wire x1="14.745" y1="27.165" x2="13.97" y2="27.94" width="0.4064" layer="16"/>
 <wire x1="13.97" y1="27.94" x2="13.97" y2="28.575" width="0.4064" layer="16"/>
-<contactref element="C2" pad="1"/>
+<contactref element="C5" pad="+"/>
+<contactref element="JP7" pad="1"/>
+<contactref element="JP7" pad="3"/>
+<contactref element="JP7" pad="5"/>
+<contactref element="JP7" pad="7"/>
+<contactref element="JP7" pad="9"/>
 </signal>
 <signal name="D8">
@@
 <contactref element="PWR" pad="A"/>
 <contactref element="R1.1" pad="1"/>
-<wire x1="47.625" y1="21.905" x2="45.185" y2="21.905" width="0.6096" layer="1"/>
-<wire x1="45.185" y1="21.905" x2="45.085" y2="22.005" width="0.6096" layer="1"/>
+<wire x1="35.78" y1="2.54" x2="35.78" y2="4.98" width="0.4064" layer="1"/>
+<wire x1="35.78" y1="4.98" x2="35.88" y2="5.08" width="0.4064" layer="1"/>
 </signal>
 <signal name="+5V/2">
@@
 <wire x1="33.915" y1="12.325" x2="33.02" y2="11.43" width="1.27" layer="1"/>
 <wire x1="33.02" y1="11.43" x2="33.02" y2="3.81" width="1.27" layer="1"/>
-<contactref element="C3" pad="1"/>
-<wire x1="36.83" y1="4.445" x2="33.655" y2="4.445" width="0.6096" layer="1"/>
-<wire x1="33.655" y1="4.445" x2="33.02" y2="3.81" width="0.6096" layer="1"/>
+<contactref element="C4" pad="+"/>
+<wire x1="37.87" y1="9.525" x2="37.87" y2="12.2" width="1.27" layer="1"/>
+<wire x1="37.87" y1="12.2" x2="37.745" y2="12.325" width="1.27" layer="1"/>
 </signal>
 <signal name="N$17">
